Commit message: [ADD] IRB 460: stylized parts for the view without the CAD model
models/irb460_110_240/stylized/: low polygon shapes with the outline and the
size of the parts of the ABB CAD model (cells of each part replaced by their
convex hulls), about 350 KB, used by the URDF in place of the boxes; the CAD
meshes, when built, still replace them. build_stylized.py builds them from the
CAD meshes.

Co-Authored-By: Claude Opus 5.5 <noreply@anthropic.com>

File: models/irb460_110_240.urdf (robot description, URDF)
Before this commit: robot irb460_110_240, 13 links, 12 joints
Links:
- link base_link: geometry visual mesh filename=package://irb460_110_240/stylized/foot.stl scale=0.001 0.001 0.001
- link link_1: geometry visual mesh filename=package://irb460_110_240/stylized/swing.stl scale=0.001 0.001 0.001
- link link_2: geometry visual mesh filename=package://irb460_110_240/stylized/lower_arm.stl scale=0.001 0.001 0.001
- link link_3: geometry visual mesh filename=package://irb460_110_240/stylized/upper_arm.stl scale=0.001 0.001 0.001
- link link_4: geometry visual mesh filename=package://irb460_110_240/stylized/tilt.stl scale=0.001 0.001 0.001
- link link_6: geometry visual mesh filename=package://irb460_110_240/stylized/disk.stl scale=0.001 0.001 0.001
- link link_plate: geometry visual mesh filename=package://irb460_110_240/stylized/link_plate.stl scale=0.001 0.001 0.001
- link lower_link: geometry visual mesh filename=package://irb460_110_240/stylized/lower_link.stl scale=0.001 0.001 0.001
- link p_arm: geometry visual mesh filename=package://irb460_110_240/stylized/p_arm.stl scale=0.001 0.001 0.001
- link p_link: geometry visual mesh filename=package://irb460_110_240/stylized/p_link.stl scale=0.001 0.001 0.001
- link upper_link: geometry visual mesh filename=package://irb460_110_240/stylized/upper_link.stl scale=0.001 0.001 0.001
