Commit message: [CHANGE] osj6: modular kit to print (CadQuery), the model generated from the parts
examples/osj6/cad/parts.py draws the parts of osj6 with CadQuery (STEP and STL): equal
pieces with a flat and a 45 degree face, spacers, base, tool flange, all with the same
interface; printed slewing rings with 6 mm balls (gothic, V or round groove) and an
internal gear of module 1 that meshes with the LEGO gears (12 teeth, ratio 5:1, motor
axle 3 LEGO holes from the axis); brackets for the LEGO Medium Angular Motor (dimensions
and pin holes from its LDraw model) and for a NEMA 14 stepper. The spacers of each arm
are parameters (SHOULDER_SPACERS, MODULE_SPACERS, WRIST_SPACERS).

build_model.py writes models/osj6.urdf from the same robot: the joint frames, the meshes
of each link and the masses of the parts (2.7 kg): the simulation and the kit are the same
robot (tube of 100 mm, 770 mm high). It replaces models/osj6/build.py (tube of 80 mm, N20
motors). The demo, the test and the README follow the new geometry; the torques show that
the LEGO motors are too weak for the axes 2 - 4 of the whole arm.

The hatch environment cad (cadquery, numpy, ocp_vscode, ocp_viewer) is separate from the
dependencies of the project; show.py shows the parts in the OCP CAD Viewer (VS Code or
the browser, hatch run cad:viewer).

Co-Authored-By: Claude Opus 5.5 <noreply@anthropic.com>

File: models/osj6.urdf (robot description, URDF)
Before this commit: robot osj6, 9 links, 8 joints
Links:
- link base_link: mass 0.2237 -> 0.3348; geometry visual mesh filename=package://osj6/parts/base_link_bracket.stl scale=0.001 0.001 0.001; visual mesh filename=package://osj6/parts/base_link_motor.stl scale=0.001 0.001 0.001
- link link_1: mass 0.1636 -> 0.3516; geometry visual mesh filename=package://osj6/parts/link_1_bracket.stl scale=0.001 0.001 0.001; visual mesh filename=package://osj6/parts/link_1_motor.stl scale=0.001 0.001 0.001
- link link_2: mass 0.2024 -> 0.4884; geometry visual mesh filename=package://osj6/parts/link_2_bracket.stl scale=0.001 0.001 0.001; visual mesh filename=package://osj6/parts/link_2_motor.stl scale=0.001 0.001 0.001
- link link_3: mass 0.2024 -> 0.4884; geometry visual mesh filename=package://osj6/parts/link_3_bracket.stl scale=0.001 0.001 0.001; visual mesh filename=package://osj6/parts/link_3_motor.stl scale=0.001 0.001 0.001
- link link_4: mass 0.2024 -> 0.4884; geometry visual mesh filename=package://osj6/parts/link_4_bracket.stl scale=0.001 0.001 0.001; visual mesh filename=package://osj6/parts/link_4_motor.stl scale=0.001 0.001 0.001
- link link_5: mass 0.1629 -> 0.4652; geometry visual mesh filename=package://osj6/parts/link_5_bracket.stl scale=0.001 0.001 0.001; visual mesh filename=package://osj6/parts/link_5_motor.stl scale=0.001 0.001 0.001
- link link_6: mass 0.0445 -> 0.0801; geometry visual mesh filename=package://osj6/parts/link_6_print.stl scale=0.001 0.001 0.001; visual mesh filename=package://osj6/parts/link_6_ring.stl scale=0.001 0.001 0.001
Joints:
- joint joint_1: limit lower=-2.9671 upper=2.9671 effort=0 velocity=1.0472 -> lower=-3.14159265 upper=3.14159265 effort=0 velocity=1.0; origin xyz=0 0 0.07 rpy=0 0 0 -> xyz=0 0 0.077 rpy=0 0 0
- joint joint_2: limit lower=-2.9671 upper=2.9671 effort=0 velocity=1.0472 -> lower=-3.14159265 upper=3.14159265 effort=0 velocity=1.0; origin xyz=0 0 0.08 rpy=0.785398163 0 0 -> xyz=0 -0.00494974747 0.0819497475 rpy=0.785398163 0 0
- joint joint_3: limit lower=-2.9671 upper=2.9671 effort=0 velocity=1.0472 -> lower=-3.14159265 upper=3.14159265 effort=0 velocity=1.0; origin xyz=0 0.0848528137 0.0848528137 rpy=1.57079633 0 3.14159265 -> xyz=0 0.105994949 0.105994949 rpy=1.57079633 0 -3.14159265
- joint joint_4: limit lower=-2.9671 upper=2.9671 effort=0 velocity=1.0472 -> lower=-3.14159265 upper=3.14159265 effort=0 velocity=1.0; origin xyz=0 0.0848528137 0.0848528137 rpy=1.57079633 0 3.14159265 -> xyz=0 0.105994949 0.105994949 rpy=1.57079633 0 -3.14159265
- joint joint_5: limit lower=-2.9671 upper=2.9671 effort=0 velocity=1.0472 -> lower=-3.14159265 upper=3.14159265 effort=0 velocity=1.0; origin xyz=0 0.0848528137 0.0848528137 rpy=1.57079633 0 3.14159265 -> xyz=0 0.105994949 0.105994949 rpy=1.57079633 0 -3.14159265
- joint joint_6: limit lower=-2.9671 upper=2.9671 effort=0 velocity=1.0472 -> lower=-3.14159265 upper=3.14159265 effort=0 velocity=1.0; origin xyz=0 0.0565685425 0.0565685425 rpy=-0.785398163 0 0 -> xyz=0 0.096873629 0.103873629 rpy=-0.785398163 0 0
- joint joint_6-tool0: origin xyz=0 0 0.01 rpy=0 0 -3.14159265 -> xyz=0 0 0.019 rpy=0 0 3.14159265
